File: hardware/P1Link.kicad_pcb (KiCad board)
At the start: 2 copper layers, 47.3 x 23.7 mm, 48 parts, among them J1 RJ12, J2 SIM_Card_Shielded, Q1 Q_NPN_CBE, Q2 Q_PMOS_GSD, Q3 Q_NMOS_GSD, U1 ZD8028C, U4 USBLC6-2SC6, U6 CH32V006F8U6, U7 ZD25WQ16C, U8 BC66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

Commit message: V0.1 finished
Parts:
- removed C10: 0.1u, Capacitor_SMD:C_0402_1005Metric
- removed C15: 10u, Capacitor_SMD:C_0402_1005Metric
- added TP5: 5V, TestPoint:TestPoint_Pad_D1.0mm, B.Cu at (44.0, 42.6)
- added TP8: 3V3, TestPoint:TestPoint_Pad_D1.0mm, B.Cu at (57.5, 50.9)
- added TP9: GND, TestPoint:TestPoint_Pad_D1.0mm, B.Cu at (60.2, 50.9)
- C3, C4, C5, R9, U4: moved to B.Cu
- C6: footprint Capacitor_SMD:C_0402_1005Metric -> Capacitor_SMD:C_1206_3216Metric
- L1: value L -> 4.7u
- Q1: value Q_NPN_CBE -> Q_NPN_BEC
- R1: value R -> 261k
- R10: value R -> 100m
- R2: value R -> 59k
- R3, R4: moved to F.Cu
- moved R11 29.6 mm to (50.2, 50.5)
- moved TH1 29.6 mm to (51.2, 50.5)
- moved TP3 27.8 mm to (64.3, 50.5)
- moved TP7 26.7 mm to (41.8, 42.0)
- moved TP2 23.3 mm to (64.3, 54.5)
- moved TP1 22.7 mm to (64.3, 52.5)
- moved C12 18.9 mm to (49.0, 40.3), turned to 135 degrees
- moved C11 18.6 mm to (46.4, 40.5), turned to 45 degrees
- moved TP4 17.6 mm to (46.4, 52.0)
- moved Y1 16.7 mm to (47.6, 41.8), turned to -135 degrees
- moved TP12 15.0 mm to (64.3, 56.5)
- moved C4 13.0 mm to (49.4, 36.4), turned to 90 degrees
- moved R4 11.6 mm to (47.0, 56.3), turned to 0 degrees
- moved C3 11.4 mm to (50.3, 36.4), turned to 90 degrees
- moved R3 11.4 mm to (47.0, 57.2), turned to 0 degrees
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Connections:
- Q1 pad 1: Net-(Q1-C) -> Net-(Q1-B)
- Q1 pad 2: Net-(Q1-B) -> GND
- Q1 pad 3: GND -> Net-(Q1-C)
- R8 pad 1: VCC -> +3V3
- U6 pad 10: unconnected-(U6-PC3-Pad10) -> /NOR_CS
- U6 pad 8: /NOR_CS -> /SIM_RESET
- U6 pad 9: unconnected-(U6-PC2-Pad9) -> /SIM_BOOT
Routing:
- net +3V3: track 8.06 -> 73.3 mm, vias 0 -> 4
- net +5V: track 6.00 -> 44.1 mm, vias 0 -> 1
- net GND: track 1.74 -> 39.4 mm, vias 0 -> 19
- net /SIM_BOOT: track 0.00 -> 23.2 mm, vias 0 -> 1
- net /P1_REQ: track 0.00 -> 22.3 mm, vias 0 -> 2
- net Net-(U8-TXD_DBG): track 0.00 -> 19.6 mm, vias 0 -> 1
- net Net-(U8-RXD_DBG): track 0.00 -> 17.1 mm, vias 0 -> 1
- net /NOR_CS: track 0.00 -> 15.3 mm, vias 0 -> 2
- net /LED: track 0.00 -> 14.5 mm, vias 0 -> 2
- net /P1_REQ_: track 0.00 -> 14.2 mm
- net /SIM_TX: track 1.20 -> 15.4 mm, vias 0 -> 1
- net /SIM_RX: track 1.26 -> 15.4 mm, vias 0 -> 1
- net Net-(U8-NETLIGHT): track 0.00 -> 13.5 mm, vias 0 -> 1
- net /P1_DAT: track 0.00 -> 12.3 mm, vias 0 -> 2
- net Net-(J1-Pad5): track 0.00 -> 11.6 mm
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Other:
- board text added: "P1Link"
- board text added: "v0.1"
