File: hardware/P1Link.kicad_sch (KiCad schematic)
At the start: 48 parts, among them J1 RJ12, J2 SIM_Card_Shielded, Q1 Q_NPN_CBE, Q2 Q_PMOS_GSD, Q3 Q_NMOS_GSD, U1 ZD8028C, U4 USBLC6-2SC6, U6 CH32V006F8U6, U7 ZD25WQ16C, U8 BC66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

Commit message: V0.1 finished
Parts:
- removed C10: 0.1u, Capacitor_SMD:C_0402_1005Metric, symbol Device:C
- removed C15: 10u, Capacitor_SMD:C_0402_1005Metric, symbol Device:C
- removed Q1: Q_NPN_CBE, Package_TO_SOT_SMD:SOT-23, symbol Transistor_BJT:Q_NPN_CBE
- added Q1: Q_NPN_BEC, Package_TO_SOT_SMD:SOT-23, symbol Transistor_BJT:Q_NPN_BEC
- added TP5: 5V, TestPoint:TestPoint_Pad_D1.0mm, symbol Connector:TestPoint
- added TP8: 3V3, TestPoint:TestPoint_Pad_D1.0mm, symbol Connector:TestPoint
- added TP9: GND, TestPoint:TestPoint_Pad_D1.0mm, symbol Connector:TestPoint
- AE1, TP1, TP12, TP2, TP3, TP4, TP6, TP7: now left out of the parts list
- C13: value 0.1u -> 100n
- C6: footprint Capacitor_SMD:C_0402_1005Metric -> Capacitor_SMD:C_1206_3216Metric
- D1: JLCPCB Part# (none) -> C965555
- J1: JLCPCB Part# (none) -> C77859; LCSC C77859 -> (none)
- J2: JLCPCB Part# (none) -> C720512
- L1: value L -> 4.7u
- Q2: JLCPCB Part# (none) -> C5261052; LCSC C5261052 -> (none)
- Q3: JLCPCB Part# (none) -> C4748714; LCSC C4748714 -> (none)
- R1: value R -> 261k
- R10: value R -> 100m; JLCPCB Part# (none) -> C1882657
- R2: value R -> 59k
- TH1: JLCPCB Part# (none) -> C89601; LCSC C77131 -> (none)
- U1: JLCPCB Part# (none) -> C2928932; LCSC C2928932 -> (none)
- U4: JLCPCB Part# (none) -> C2687116; LCSC C2687116 -> (none)
- U6: JLCPCB Part# (none) -> C42431288; LCSC C42431288 -> (none)
- U7: JLCPCB Part# (none) -> C7304007; LCSC C7304007 -> (none)
- U8: JLCPCB Part# (none) -> C5140591
- Y1: JLCPCB Part# (none) -> C2965580; LCSC C2965580 -> (none)
Connections:
- net VCC is gone; now on net +3V3: R8.1
- net +3V3: now also TP8.1
- net +5V: now also TP5.1
- net GND: now also Q1.2 (E), TP9.1
- net NOR_CS: now also U6.10 (PC3); no longer U6.8 (PC1)
- net SIM_BOOT: now also U6.9 (PC2)
- net SIM_RESET: now also U6.8 (PC1)
- net at R6.2: now also Q1.1 (B)
- net at Q2.1 (G), R7.1: now also Q1.3 (C)
Other:
- note added: "<0.5A"
- note removed: "T1CH3"
- note removed: "TODO ESD"
- note removed: "TODO bulk"
- note removed: "TODO testpoints"
- note removed: "~0.5A"
- moved on the sheet: TP4, U6
